Commit message: Update rv_4frl_d.urdf.xacro

File: src/mitsubishi_ros2_description/urdf/rv_4frl_d/rv_4frl_d.urdf.xacro (robot description, xacro)
@@ -139,5 +139,5 @@
       </visual>
       <collision>
-        <origin xyz="-0.0498 0 -0.525" rpy="1.57079633 0 0" />
+        <origin xyz="0 0 ${-0.350-0.310-0.050}" rpy="1.57079633 0 0" />
         <geometry>
           <mesh filename="file://$(find mitsubishi_ros2_description)/meshes/rv_4frl_d/RV-4FRL_05_NO2ARM.stl" scale="0.001 0.001 0.001"/>
@@ -168,5 +168,5 @@
       </visual>
       <collision>
-        <origin xyz="-0.0498 -0.795 0" rpy="0 0 0" />
+        <origin xyz="0.335 ${-0.350-0.310-0.050} 0.0 " rpy="0 0 0" />
         <geometry>
           <mesh filename="file://$(find mitsubishi_ros2_description)/meshes/rv_4frl_d/RV-4FRL_06_WRIST.stl" scale="0.001 0.001 0.001"/>
@@ -196,5 +196,5 @@
       </visual>
       <collision>
-        <origin xyz="-0.05 -0.05 -0.795" rpy="1.5 0 0" />
+        <origin xyz="${0.335+0.08} ${-0.350-0.310-0.050} 0" rpy="0 0 0" />
         <geometry>
           <mesh filename="file://$(find mitsubishi_ros2_description)/meshes/rv_4frl_d/RV-4FRL_07_HAND_FLANGE.stl" scale="0.001 0.001 0.001"/>
@@ -214,3 +214,39 @@
     </joint>
   </xacro:macro>
+  <xacro:include filename="$(find mitsubishi_ros2_description)/urdf/realsense2.urdf.xacro" />
+  <!-- <link name="world" /> -->
+  <!-- <joint name="world_joint" type="fixed">
+    <parent link="world" />
+    <child link = "base_link" />
+    <origin xyz="0.0 0.0 0.0" rpy="0.0 0.0 0.0" />
+  </joint> -->
+  <joint name="realsense_joint" type="fixed">
+    <parent link="rv_4frl_d_base_link" />
+    <child link="camera_link" />
+      <origin xyz="1.152 0.02 1.2379" rpy="0.0 0.8342674 3.14" />
+  </joint>
+  <!-- <joint name="realsense_joint" type="fixed">
+    <parent link="wrist_2_link" />
+    <child link="camera_link" />
+    <origin xyz="0.0 0.05 0.08" rpy="0.0 0.0 1.57" />
+  </joint> -->
+  <link name="camera_link">
+  <collision>
+    <origin xyz="0 0 0" rpy="0 0 0"/>
+    <geometry>
+      <box size="0.001 0.001 0.001"/>
+    </geometry>
+  </collision>
+  <visual>
+    <origin xyz="0 0 0" rpy="1.57 0 1.57"/>
+    <geometry>
+        <mesh filename="file://$(find mitsubishi_ros2_description)/meshes/NAVRS.STL" />
+    </geometry>
+  </visual>
+  <inertial>
+    <mass value="1e-5" />
+    <origin xyz="0 0 0" rpy="0 0 0"/>
+    <inertia ixx="0" ixy="0" ixz="0" iyy="0" iyz="0" izz="0" />
+  </inertial>
+  </link>
 </robot>

Commit message: Update rv_4frl_d.urdf.xacro
Noticed a little error for rv_4frl_d  urdf collision while working on a school project which would later be implemented on real robot

File: src/mitsubishi_ros2_description/urdf/rv_4frl_d/rv_4frl_d.urdf.xacro (robot description, xacro)
@@ -214,39 +214,3 @@
     </joint>
   </xacro:macro>
-  <xacro:include filename="$(find mitsubishi_ros2_description)/urdf/realsense2.urdf.xacro" />
-  <!-- <link name="world" /> -->
-  <!-- <joint name="world_joint" type="fixed">
-    <parent link="world" />
-    <child link = "base_link" />
-    <origin xyz="0.0 0.0 0.0" rpy="0.0 0.0 0.0" />
-  </joint> -->
-  <joint name="realsense_joint" type="fixed">
-    <parent link="rv_4frl_d_base_link" />
-    <child link="camera_link" />
-      <origin xyz="1.152 0.02 1.2379" rpy="0.0 0.8342674 3.14" />
-  </joint>
-  <!-- <joint name="realsense_joint" type="fixed">
-    <parent link="wrist_2_link" />
-    <child link="camera_link" />
-    <origin xyz="0.0 0.05 0.08" rpy="0.0 0.0 1.57" />
-  </joint> -->
-  <link name="camera_link">
-  <collision>
-    <origin xyz="0 0 0" rpy="0 0 0"/>
-    <geometry>
-      <box size="0.001 0.001 0.001"/>
-    </geometry>
-  </collision>
-  <visual>
-    <origin xyz="0 0 0" rpy="1.57 0 1.57"/>
-    <geometry>
-        <mesh filename="file://$(find mitsubishi_ros2_description)/meshes/NAVRS.STL" />
-    </geometry>
-  </visual>
-  <inertial>
-    <mass value="1e-5" />
-    <origin xyz="0 0 0" rpy="0 0 0"/>
-    <inertia ixx="0" ixy="0" ixz="0" iyy="0" iyz="0" izz="0" />
-  </inertial>
-  </link>
 </robot>
